File: PantryLights/PantryLights.kicad_sch (KiCad schematic)
At the start: 43 parts, among them J1 Barrel_Jack_Switch, J2 8P8C_LED_Shielded, J3 Conn_01x04, J4 Conn_01x04, Q1 IRF540N, Q2 IRF540N, SW1 SW_MEC_5E, SW2 SW_MEC_5E, SW3 SW_MEC_5E, SW4 SW_MEC_5E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

Commit message: Added Gerbers per REV_1
Parts:
- added C9: 100n, Capacitor_SMD:C_0603_1608Metric_Pad1.08x0.95mm_HandSolder, symbol Device:C
- added J5: Conn_02x03_Counter_Clockwise, Connector_PinHeader_2.54mm:PinHeader_2x03_P2.54mm_Vertical, symbol Connector_Generic:Conn_02x03_Counter_Clockwise
- added R11: 220R, Resistor_SMD:R_0603_1608Metric_Pad0.98x0.95mm_HandSolder, symbol Device:R_US
Connections:
- net +5V: now also C9.2, J5.2 (Pin_2)
- net GND: now also J2.SH, C9.1, J5.6 (Pin_6)
- net MISO: now also J5.1 (Pin_1)
- net MOSI: now also J5.4 (Pin_4)
- net RESET: now also J5.5 (Pin_5)
- net SCK: now also J5.3 (Pin_3)
- net at J4.1 (Pin_1), R6.1, TP4.1: now also U1.24 (PC1); no longer U1.23 (PC0)
- net at J4.3 (Pin_3), R5.2, TP5.1: now also U1.23 (PC0); no longer U1.24 (PC1)
- net at D5.2 (A), TP3.1, U1.13 (PB1): now also R11.1; no longer Q1.1 (G), Q2.1 (G)
- new net: Q1.1 (G), Q2.1 (G), R11.2
Other:
- moved on the sheet: D5, R7, TP3
