File: PantryLights/PantryLights.kicad_pcb (KiCad board)
At the start: 2 copper layers, 78.7 x 52.1 mm, 43 parts, among them J1 Barrel_Jack_Switch, J2 8P8C_LED_Shielded, J3 Conn_01x04, J4 Conn_01x04, Q1 IRF540N, Q2 IRF540N, SW1 SW_MEC_5E, SW2 SW_MEC_5E, SW3 SW_MEC_5E, SW4 SW_MEC_5E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

Commit message: Added Gerbers per REV_1
Parts:
- added C9: 100n, Capacitor_SMD:C_0603_1608Metric_Pad1.08x0.95mm_HandSolder, F.Cu at (153.7, 114.3)
- added J5: Conn_02x03_Counter_Clockwise, Connector_PinHeader_2.54mm:PinHeader_2x03_P2.54mm_Vertical, F.Cu at (130.8, 91.5)
- added R11: 220R, Resistor_SMD:R_0603_1608Metric_Pad0.98x0.95mm_HandSolder, F.Cu at (121.3, 104.1)
- moved TP3 16.1 mm to (121.9, 100.3)
- moved TP2 11.8 mm to (108.6, 101.6)
- moved TP4 8.47 mm to (157.5, 109.2)
- moved R9 6.86 mm to (138.4, 90.3), turned to 0 degrees
- moved R8 6.13 mm to (138.5, 83.0), turned to 0 degrees
- moved J1 6.01 mm to (117.4, 84.5)
- moved R10 5.95 mm to (138.4, 96.9), turned to 0 degrees
- moved U2 4.73 mm to (117.5, 94.6)
- moved R1 3.63 mm to (165.1, 75.3), turned to -90 degrees
- moved R2 3.23 mm to (165.1, 87.7), turned to -90 degrees
- moved C3 2.85 mm to (111.5, 99.1)
- moved C2 2.83 mm to (118.8, 99.1)
- moved D3 1.44 mm to (138.4, 87.3)
- moved D2 1.00 mm to (138.4, 93.8)
- moved D4 1.00 mm to (138.4, 79.9)
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Connections:
- J2 pad SH: unconnected-(J2-PadSH) -> GND
- J4 pad 1: Net-(U1-Pad23) -> Net-(J4-Pad1)
- J4 pad 3: Net-(U1-Pad24) -> Net-(J4-Pad3)
- Q1 pad 1: Net-(U1-Pad13) -> Net-(Q1-Pad1)
- Q2 pad 1: Net-(U1-Pad13) -> Net-(Q1-Pad1)
- R5 pad 2: Net-(U1-Pad24) -> Net-(J4-Pad3)
- R6 pad 1: Net-(U1-Pad23) -> Net-(J4-Pad1)
- TP4 pad 1: Net-(U1-Pad23) -> Net-(J4-Pad1)
- TP5 pad 1: Net-(U1-Pad24) -> Net-(J4-Pad3)
- U1 pad 23: Net-(U1-Pad23) -> Net-(J4-Pad3)
- U1 pad 24: Net-(U1-Pad24) -> Net-(J4-Pad1)
Routing:
- net +5V: track 0.00 -> 231.2 mm, vias 0 -> 6
- net RESET: track 0.00 -> 92.2 mm, vias 0 -> 1
- net +12V: track 0.00 -> 69.4 mm
- net RX: track 0.00 -> 59.4 mm, vias 0 -> 1
- net TX: track 0.00 -> 58.4 mm, vias 0 -> 1
- net Net-(U1-Pad2): track 0.00 -> 58.4 mm, vias 0 -> 2
- net Net-(J4-Pad3): track 0.00 -> 56.1 mm
- net Net-(U1-Pad1): track 0.00 -> 47.1 mm, vias 0 -> 2
- net Net-(J4-Pad1): track 0.00 -> 40.9 mm
- net Net-(U1-Pad13): track 0.00 -> 39.7 mm
- net Net-(U1-Pad32): track 0.00 -> 35.6 mm, vias 0 -> 1
- net Net-(U1-Pad9): track 0.00 -> 32.1 mm
- net MISO: track 0.00 -> 27.6 mm, vias 0 -> 1
- net Net-(U1-Pad10): track 0.00 -> 24.3 mm
- net SCK: track 0.00 -> 23.8 mm, vias 0 -> 1
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- added copper zone on B.Cu, net GND
- added copper zone on F.Cu, net GND
Other:
- rule pad_to_mask_clearance: 0 -> 0.0508
- board text added: "Jan 26, 2022 Pantry Lighting REV 1"

Commit message: Second PCB Revision
Parts:
- added C10: 100n, Capacitor_SMD:C_0603_1608Metric_Pad1.08x0.95mm_HandSolder, F.Cu at (153.2, 97.8)
- added R12: 1K, Resistor_SMD:R_0603_1608Metric_Pad0.98x0.95mm_HandSolder, F.Cu at (145.5, 87.5)
- added R13: 1K, Resistor_SMD:R_0603_1608Metric_Pad0.98x0.95mm_HandSolder, F.Cu at (145.5, 89.6)
- added R14: 1M, Resistor_SMD:R_0603_1608Metric_Pad0.98x0.95mm_HandSolder, F.Cu at (131.0, 94.7)
- J3, J4: footprint TerminalBlock_Phoenix:TerminalBlock_Phoenix_MKDS-1,5-4-5.08_1x04_P5.08mm_Horizontal -> Personal:TerminalBlock_Right-Angle_Modular-1,5-4-5.08_1x04_P5.08mm_Horizontal
- Y1: footprint Crystal:Crystal_HC49-4H_Vertical -> Crystal:Crystal_SMD_3225-4Pin_3.2x2.5mm_HandSoldering
- moved SW4 39.8 mm to (138.1, 76.8), turned to -90 degrees
- moved Y1 33.3 mm to (127.8, 98.0), turned to -90 degrees
- moved C6 32.6 mm to (129.2, 89.8), turned to 180 degrees
- moved J5 31.5 mm to (154.9, 111.6), turned to 90 degrees
- moved C4 30.8 mm to (128.3, 94.0), turned to 0 degrees
- moved TP2 28.2 mm to (123.2, 77.5)
- moved J4 27.9 mm to (133.3, 111.8)
- moved TP5 27.6 mm to (148.6, 104.1)
- moved R5 26.6 mm to (144.6, 104.3), turned to 0 degrees
- moved C8 25.1 mm to (145.5, 91.7), turned to 180 degrees
- moved TP4 24.7 mm to (133.3, 104.1)
- moved R4 23.2 mm to (145.5, 96.1), turned to 180 degrees
- moved U1 22.7 mm to (137.2, 91.4), turned to 0 degrees
- moved R6 22.5 mm to (138.5, 104.3), turned to 0 degrees
- moved C9 22.0 mm to (145.5, 93.9)
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Connections:
- net Net-(J4-Pad1) renamed /PHOTORESISTOR_IN
- net Net-(J4-Pad3) renamed /DOOR_SW_IN
- net Net-(Q1-Pad1) renamed /LIGHTS_CL
- net Net-(U1-Pad1) renamed /BTN_2
- net Net-(U1-Pad13) renamed /LIGHT_SIGNAL
- net Net-(U1-Pad2) renamed /BTN_3
- net Net-(U1-Pad32) renamed /BTN_1
- C4 pad 2: Net-(Y1-Pad2) -> /OSC_A
- C5 pad 2: Net-(Y1-Pad1) -> /OSC_B
- D2 pad 1: Net-(D2-Pad1) -> GND
- D2 pad 2: Net-(U1-Pad11) -> Net-(R10-Pad2)
- D3 pad 1: Net-(D3-Pad1) -> GND
- D3 pad 2: Net-(U1-Pad10) -> Net-(R9-Pad2)
- D4 pad 1: Net-(D4-Pad1) -> GND
- D4 pad 2: Net-(U1-Pad9) -> Net-(R8-Pad2)
- J2 pad 11: TX -> Net-(J2-Pad11)
- J2 pad 3: TX -> Net-(J2-Pad11)
- J2 pad 6: RX -> Net-(J2-Pad6)
- J2 pad 7: unconnected-(J2-Pad7) -> Net-(C10-Pad1)
- J2 pad 9: RX -> Net-(J2-Pad6)
- R10 pad 1: Net-(D2-Pad1) -> /LED_3
- R10 pad 2: GND -> Net-(R10-Pad2)
- R8 pad 1: Net-(D4-Pad1) -> /LED_1
- R8 pad 2: GND -> Net-(R8-Pad2)
- R9 pad 1: Net-(D3-Pad1) -> /LED_2
- R9 pad 2: GND -> Net-(R9-Pad2)
- U1 pad 10: Net-(U1-Pad10) -> /LED_2
- U1 pad 11: Net-(U1-Pad11) -> /LED_3
- U1 pad 7: Net-(Y1-Pad2) -> /OSC_A
- U1 pad 8: Net-(Y1-Pad1) -> /OSC_B
- U1 pad 9: Net-(U1-Pad9) -> /LED_1
- Y1 pad 1: Net-(Y1-Pad1) -> /OSC_A
- Y1 pad 2: Net-(Y1-Pad2) -> GND
Routing:
- net +5V: track 231.2 -> 142.3 mm, vias 6 -> 2
- net RX: track 59.4 -> 12.2 mm, vias 1 -> 0
- net TX: track 58.4 -> 12.8 mm, vias 1 -> 0
- net RESET: track 92.2 -> 58.9 mm
- net Net-(U1-Pad9): track 32.1 -> 0.00 mm
- net Net-(U1-Pad10): track 24.3 -> 0.00 mm
- net GND: track 23.6 -> 0.00 mm, vias 52 -> 0
- net /DOOR_SW_IN: track 56.1 -> 32.8 mm, vias 0 -> 2
- net Net-(Y1-Pad2): track 22.1 -> 0.00 mm
- net Net-(Y1-Pad1): track 17.7 -> 0.00 mm
- net Net-(U1-Pad11): track 17.6 -> 0.00 mm
- net /BTN_1: track 35.6 -> 18.7 mm, vias 1 -> 0
- net MOSI: track 19.7 -> 35.7 mm, vias 1 -> 0
- net /BTN_3: track 58.4 -> 42.9 mm, vias 2 -> 0
- net /BTN_2: track 47.1 -> 32.0 mm, vias 2 -> 0
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- removed copper zone on B.Cu, net GND
- removed copper zone on F.Cu, net GND
Other:
- board outline removed
- rule pad_to_mask_clearance: 0.0508 -> 0
- board text removed: "Jan 26, 2022 Pantry Lighting REV 1"

Commit message: Board Order
Parts:
- added C11: 4.7u, Capacitor_SMD:C_1206_3216Metric_Pad1.33x1.80mm_HandSolder, F.Cu at (128.6, 96.8)
- moved R7 15.0 mm to (131.2, 98.1), turned to -90 degrees
- moved R11 13.1 mm to (134.2, 98.6)
- moved R12 12.3 mm to (157.2, 91.2)
- moved R13 12.3 mm to (157.2, 93.3)
- moved C8 12.3 mm to (157.2, 95.4)
- moved C9 12.3 mm to (157.2, 97.6)
- moved R4 12.3 mm to (157.2, 99.8), turned to 0 degrees
- moved D2 12.1 mm to (158.6, 105.2)
- moved R10 12.1 mm to (158.6, 103.4)
- moved D3 12.1 mm to (152.2, 105.2)
- moved D4 12.1 mm to (145.9, 105.2)
- moved R8 12.1 mm to (145.9, 103.4)
- moved R9 12.1 mm to (152.2, 103.4)
- moved C5 11.9 mm to (142.4, 102.9)
- moved C6 11.9 mm to (140.5, 93.7)
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Routing:
- net GND: track 0.00 -> 123.1 mm, vias 0 -> 50
- net Net-(J2-Pad11): track 0.00 -> 39.5 mm
- net +5V: track 142.3 -> 165.8 mm, vias 2 -> 3
- net Net-(J2-Pad6): track 0.00 -> 21.8 mm
- net +12V: track 64.5 -> 57.9 mm
- net Net-(J2-Pad12): track 0.00 -> 2.81 mm
- net Net-(J2-Pad10): track 0.00 -> 2.75 mm
- net RESET: track 58.9 -> 60.9 mm, vias 1 -> 3
- net /DOOR_SW_IN: track 32.8 -> 31.1 mm
- net /PHOTORESISTOR_IN: track 28.8 -> 27.1 mm
- net /LIGHTS_CL: track 24.5 -> 23.0 mm
- net /LIGHT_SIGNAL: track 31.9 -> 32.5 mm
- net RX: track 12.2 -> 12.8 mm
- net TX: track 12.8 -> 13.4 mm
- net /OSC_B: track 8.43 -> 7.92 mm
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- added copper zone on F.Cu, net +12V
- added copper zone on F.Cu, net +5V
- added copper zone on B.Cu, net GND
- added copper zone on F.Cu, net GND
Other:
- board outline added: 70 x 40 mm
- board text added: "+12V"
- board text added: "+5V"
- board text added: "-"
- board text added: "B1"
- board text added: "B2"
- board text added: "B3"
- board text added: "CRYSTAL OSC"
- board text added: "D"
- board text added: "DOOR"
- board text added: "DOR"
- board text added: "DTR"
- board text added: "Feb 17, 2022 Pantry Lighting REV 2"
- board text added: "G"
- board text added: "GND"
- board text added: "ICSP"
- board text added: "JLCJLCJLCJLC"
- board text added: "L1"
- board text added: "L2"
- board text added: "L3"
- board text added: "MI"
- board text added: "MO"
- board text added: "O1"
- board text added: "O2"
- board text added: "OUT"
- board text added: "OUT 1"
- board text added: "OUT 2"
- board text added: "P"
- board text added: "PHOT"
- board text added: "PHOTORSTR"
- board text added: "PWR"
- board text added: "RST"
- board text added: "RX"
- board text added: "SC"
- board text added: "SCK"
- board text added: "THE_ERCULES"
- board text added: "TX"
- board text added: "⊕"
